File: Hardware/SparkFun_LED_Array_8x7_Charlieplex.brd (EAGLE design)
At the start: 27.9 x 43.2 mm, 76 parts

Commit message: Added 'BadgerArray' to silk
Parts:
- moved U$1 0.54 mm to (7.82, 37.8)
Other:
- board text added: "BadgerArray"
Changed lines of the file:
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@@
 <setting verticaltext="up"/>
 </settings>
-<grid distance="0.05" unitdist="inch" unit="inch" style="dots" multiple="1" display="yes" altdistance="0.005" altunitdist="inch" altunit="inch"/>
+<grid distance="0.01" unitdist="inch" unit="inch" style="dots" multiple="1" display="yes" altdistance="0.005" altunitdist="inch" altunit="inch"/>
 <layers>
 <layer number="1" name="Top" color="4" fill="1" visible="yes" active="yes"/>
@@
 <wire x1="3.81" y1="0.508" x2="24.13" y2="0.508" width="0.254" layer="22"/>
 <wire x1="3.81" y1="0.254" x2="24.13" y2="0.254" width="0.254" layer="22"/>
+<text x="13.97" y="37.719" size="1.27" layer="21" font="vector" ratio="15" align="center">BadgerArray</text>
 </plain>
 <attributes>
@@
 <element name="STANDOFF1" library="SparkFun-Electromechanical" package="STAND-OFF" value="STAND-OFF" x="25.4" y="40.64" rot="R90"/>
 <element name="STANDOFF2" library="SparkFun-Electromechanical" package="STAND-OFF" value="STAND-OFF" x="2.54" y="40.64" rot="R90"/>
-<element name="U$1" library="SparkFun-Aesthetics" package="SFE_LOGO_NAME_FLAME_.1" value="SFE_LOGO_NAME_FLAME.1_INCH" x="8.001" y="37.338"/>
+<element name="U$1" library="SparkFun-Aesthetics" package="SFE_LOGO_NAME_FLAME_.1" value="SFE_LOGO_NAME_FLAME.1_INCH" x="7.8232" y="37.846"/>
 <element name="JP1" library="SparkFun-Connectors" package="1X08_LOCK_NO_SILK" value="" x="22.86" y="1.27" rot="R180"/>
 <element name="U$2" library="SparkFun-Aesthetics" package="DUMMY" value="BADGERHACK_LOGODUMMY" x="-31.75" y="-12.7"/>
